File: hardware/keyboard/keyboard.kicad_sch (KiCad schematic)
At the start: 38 parts, among them J1 Conn_01x08_Pin, J2 Conn_01x08_Pin, J3 Conn_01x08_Pin, J4 Conn_01x08_Pin, J5 Conn_01x26_Socket, J6 Conn_01x12_Pin, Q1 PC817C, Q10 PC817C, Q11 PC817C, Q12 PC817C, Q13 PC817C, Q14 PC817C, Q15 PC817C, Q16 PC817C, Q17 PC817C, Q18 PC817C, Q19 PC817C, Q2 PC817C, Q20 PC817C, Q21 PC817C, Q22 PC817C, Q23 PC817C, Q24 PC817C, Q25 PC817C, Q26 PC817C, Q27 PC817C, Q28 PC817C, Q29 PC817C, Q3 PC817C, Q30 PC817C, Q31 PC817C, Q32 PC817C, Q4 PC817C, Q5 PC817C, Q6 PC817C, Q7 PC817C, Q8 PC817C, Q9 PC817C

Commit message: Updates
Parts:
- J1, J2, J3, J4: footprint (none) -> Connector_PinHeader_1.00mm:PinHeader_1x08_P1.00mm_Vertical
- J5: footprint (none) -> Connector_PinHeader_1.00mm:PinHeader_1x26_P1.00mm_Vertical
- J6: footprint (none) -> Connector_PinHeader_1.00mm:PinHeader_1x12_P1.00mm_Vertical
Connections:
- net at Q1.2, Q2.2, Q3.2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: now also Q10.2, Q11.2, Q12.2, Q13.2, Q14.2, Q15.2, Q16.2, Q17.2, Q18.2, Q19.2, Q20.2, Q21.2, Q22.2, Q23.2, Q24.2, Q25.2, Q26.2, Q27.2, Q28.2, Q29.2, Q30.2, Q31.2, Q32.2, Q9.2
Changed lines of the file:
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@@
   (junction (at 121.92 74.93) (diameter 0) (color 0 0 0 0)
   )
+  (junction (at 157.48 140.97) (diameter 0) (color 0 0 0 0)
+  )
   (junction (at 182.88 120.65) (diameter 0) (color 0 0 0 0)
   )
@@
   (junction (at 218.44 88.9) (diameter 0) (color 0 0 0 0)
   )
+  (junction (at 34.29 140.97) (diameter 0) (color 0 0 0 0)
+  )
   (junction (at 62.23 73.66) (diameter 0) (color 0 0 0 0)
   )
@@
   (junction (at 182.88 29.21) (diameter 0) (color 0 0 0 0)
   )
+  (junction (at 96.52 140.97) (diameter 0) (color 0 0 0 0)
+  )
   (junction (at 157.48 59.69) (diameter 0) (color 0 0 0 0)
   )
@@
     (stroke (width 0) (type default))
   )
+  (wire (pts (xy 157.48 140.97) (xy 218.44 140.97))
+    (stroke (width 0) (type default))
+  )
   (wire (pts (xy 218.44 104.14) (xy 222.25 104.14))
     (stroke (width 0) (type default))
@@
     (stroke (width 0) (type default))
   )
+  (wire (pts (xy 96.52 140.97) (xy 157.48 140.97))
+    (stroke (width 0) (type default))
+  )
   (wire (pts (xy 157.48 44.45) (xy 160.02 44.45))
     (stroke (width 0) (type default))
@@
     (stroke (width 0) (type default))
   )
-  (wire (pts (xy 157.48 135.89) (xy 157.48 137.16))
+  (wire (pts (xy 157.48 135.89) (xy 157.48 140.97))
     (stroke (width 0) (type default))
   )
@@
     (stroke (width 0) (type default))
   )
-  (wire (pts (xy 34.29 134.62) (xy 34.29 137.16))
+  (wire (pts (xy 34.29 134.62) (xy 34.29 140.97))
     (stroke (width 0) (type default))
   )
@@
     (stroke (width 0) (type default))
   )
+  (wire (pts (xy 34.29 140.97) (xy 34.29 144.78))
+    (stroke (width 0) (type default))
+  )
   (wire (pts (xy 92.71 54.61) (xy 99.06 54.61))
     (stroke (width 0) (type default))
@@
     (stroke (width 0) (type default))
   )
-  (wire (pts (xy 218.44 134.62) (xy 218.44 137.16))
+  (wire (pts (xy 218.44 134.62) (xy 218.44 140.97))
     (stroke (width 0) (type default))
   )
@@
     (stroke (width 0) (type default))
   )
+  (wire (pts (xy 34.29 140.97) (xy 96.52 140.97))
+    (stroke (width 0) (type default))
+  )
   (wire (pts (xy 246.38 27.94) (xy 246.38 43.18))
     (stroke (width 0) (type default))
@@
     (stroke (width 0) (type default))
   )
-  (wire (pts (xy 96.52 135.89) (xy 96.52 137.16))
+  (wire (pts (xy 96.52 135.89) (xy 96.52 140.97))
     (stroke (width 0) (type default))
   )
@@
     )
   )
-  (symbol (lib_id "power:PWR_FLAG") (at 157.48 137.16 0) (mirror x) (unit 1)
-    (in_bom yes) (on_board yes) (dnp no)
-    (property "Reference" "#FLG03" (at 157.48 139.065 0)
-      (effects (font (size 1.27 1.27)) hide)
-    )
-    (property "Value" "PWR_FLAG" (at 157.48 140.97 0)
-      (effects (font (size 1.27 1.27)))
-    )
-    (property "Footprint" "" (at 157.48 137.16 0)
-      (effects (font (size 1.27 1.27)) hide)
-    )
-    (property "Datasheet" "~" (at 157.48 137.16 0)
-      (effects (font (size 1.27 1.27)) hide)
-    )
-    (pin "1")
-    (instances
-      (project "keyboard"
-        (path "/d630d641-5fc5-4c38-84e8-1764deeac9f2"
-          (reference "#FLG03") (unit 1)
-        )
-      )
-    )
-  )
-  (symbol (lib_id "power:PWR_FLAG") (at 96.52 137.16 0) (mirror x) (unit 1)
-    (in_bom yes) (on_board yes) (dnp no)
-    (property "Reference" "#FLG02" (at 96.52 139.065 0)
-      (effects (font (size 1.27 1.27)) hide)
-    )
-    (property "Value" "PWR_FLAG" (at 96.52 140.97 0)
-      (effects (font (size 1.27 1.27)))
-    )
-    (property "Footprint" "" (at 96.52 137.16 0)
-      (effects (font (size 1.27 1.27)) hide)
-    )
-    (property "Datasheet" "~" (at 96.52 137.16 0)
-      (effects (font (size 1.27 1.27)) hide)
-    )
-    (pin "1")
-    (instances
-      (project "keyboard"
-        (path "/d630d641-5fc5-4c38-84e8-1764deeac9f2"
-          (reference "#FLG02") (unit 1)
-        )
-      )
-    )
-  )
   (symbol (lib_id "PC817C:PC817C") (at 171.45 87.63 0) (unit 1)
     (in_bom yes) (on_board yes) (dnp no) (fields_autoplaced)
@@
       (effects (font (size 1.27 1.27)))
     )
-    (property "Footprint" "" (at 265.43 93.98 0)
+    (property "Footprint" "Connector_PinHeader_1.00mm:PinHeader_1x12_P1.00mm_Vertical" (at 265.43 93.98 0)
       (effects (font (size 1.27 1.27)) hide)
     )
@@
       (effects (font (size 1.27 1.27)))
     )
-    (property "Footprint" "" (at 80.01 80.01 0)
+    (property "Footprint" "Connector_PinHeader_1.00mm:PinHeader_1x08_P1.00mm_Vertical" (at 80.01 80.01 0)
       (effects (font (size 1.27 1.27)) hide)
     )
@@
       (effects (font (size 1.27 1.27)))
     )
-    (property "Footprint" "" (at 147.32 78.74 0)
+    (property "Footprint" "Connector_PinHeader_1.00mm:PinHeader_1x08_P1.00mm_Vertical" (at 147.32 78.74 0)
       (effects (font (size 1.27 1.27)) hide)
     )
@@
     )
   )
-  (symbol (lib_id "power:PWR_FLAG") (at 218.44 137.16 0) (mirror x) (unit 1)
-    (in_bom yes) (on_board yes) (dnp no)
-    (property "Reference" "#FLG04" (at 218.44 139.065 0)
-      (effects (font (size 1.27 1.27)) hide)
-    )
-    (property "Value" "PWR_FLAG" (at 218.44 140.97 0)
-      (effects (font (size 1.27 1.27)))
-    )
-    (property "Footprint" "" (at 218.44 137.16 0)
-      (effects (font (size 1.27 1.27)) hide)
-    )
-    (property "Datasheet" "~" (at 218.44 137.16 0)
-      (effects (font (size 1.27 1.27)) hide)
-    )
-    (pin "1")
-    (instances
-      (project "keyboard"
-        (path "/d630d641-5fc5-4c38-84e8-1764deeac9f2"
-          (reference "#FLG04") (unit 1)
-        )
-      )
-    )
-  )
   (symbol (lib_id "PC817C:PC817C") (at 109.22 102.87 0) (unit 1)
     (in_bom yes) (on_board yes) (dnp no) (fields_autoplaced)
@@
       (effects (font (size 1.27 1.27)))
     )
-    (property "Footprint" "" (at 93.98 176.53 0)
+    (property "Footprint" "Connector_PinHeader_1.00mm:PinHeader_1x26_P1.00mm_Vertical" (at 93.98 176.53 0)
       (effects (font (size 1.27 1.27)) hide)
     )
@@
     )
   )
-  (symbol (lib_id "power:PWR_FLAG") (at 34.29 137.16 0) (mirror x) (unit 1)
+  (symbol (lib_id "power:PWR_FLAG") (at 34.29 144.78 0) (mirror x) (unit 1)
     (in_bom yes) (on_board yes) (dnp no)
-    (property "Reference" "#FLG01" (at 34.29 139.065 0)
+    (property "Reference" "#FLG01" (at 34.29 146.685 0)
       (effects (font (size 1.27 1.27)) hide)
     )
-    (property "Value" "PWR_FLAG" (at 34.29 140.97 0)
+    (property "Value" "PWR_FLAG" (at 34.29 148.59 0)
       (effects (font (size 1.27 1.27)))
     )
-    (property "Footprint" "" (at 34.29 137.16 0)
+    (property "Footprint" "" (at 34.29 144.78 0)
       (effects (font (size 1.27 1.27)) hide)
     )
-    (property "Datasheet" "~" (at 34.29 137.16 0)
+    (property "Datasheet" "~" (at 34.29 144.78 0)
       (effects (font (size 1.27 1.27)) hide)
     )
@@
       (effects (font (size 1.27 1.27)))
     )
-    (property "Footprint" "" (at 207.01 80.01 0)
+    (property "Footprint" "Connector_PinHeader_1.00mm:PinHeader_1x08_P1.00mm_Vertical" (at 207.01 80.01 0)
       (effects (font (size 1.27 1.27)) hide)
     )
@@
       (effects (font (size 1.27 1.27)))
     )
-    (property "Footprint" "" (at 20.32 77.47 0)
+    (property "Footprint" "Connector_PinHeader_1.00mm:PinHeader_1x08_P1.00mm_Vertical" (at 20.32 77.47 0)
       (effects (font (size 1.27 1.27)) hide)
     )

Commit message: Update
Parts:
- J1, J2, J3, J4: footprint Connector_PinHeader_1.00mm:PinHeader_1x08_P1.00mm_Vertical -> Connector_PinHeader_2.54mm:PinHeader_1x08_P2.54mm_Vertical
- J5: footprint Connector_PinHeader_1.00mm:PinHeader_1x26_P1.00mm_Vertical -> Connector_PinHeader_2.54mm:PinHeader_1x26_P2.54mm_Vertical
- J6: footprint Connector_PinHeader_1.00mm:PinHeader_1x12_P1.00mm_Vertical -> Connector_PinHeader_2.54mm:PinHeader_1x12_P2.54mm_Vertical
Changed lines of the file:
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@@
       (effects (font (size 1.27 1.27)))
     )
-    (property "Footprint" "Connector_PinHeader_1.00mm:PinHeader_1x12_P1.00mm_Vertical" (at 265.43 93.98 0)
+    (property "Footprint" "Connector_PinHeader_2.54mm:PinHeader_1x12_P2.54mm_Vertical" (at 265.43 93.98 0)
       (effects (font (size 1.27 1.27)) hide)
     )
@@
       (effects (font (size 1.27 1.27)))
     )
-    (property "Footprint" "Connector_PinHeader_1.00mm:PinHeader_1x08_P1.00mm_Vertical" (at 80.01 80.01 0)
+    (property "Footprint" "Connector_PinHeader_2.54mm:PinHeader_1x08_P2.54mm_Vertical" (at 80.01 80.01 0)
       (effects (font (size 1.27 1.27)) hide)
     )
@@
       (effects (font (size 1.27 1.27)))
     )
-    (property "Footprint" "Connector_PinHeader_1.00mm:PinHeader_1x08_P1.00mm_Vertical" (at 147.32 78.74 0)
+    (property "Footprint" "Connector_PinHeader_2.54mm:PinHeader_1x08_P2.54mm_Vertical" (at 147.32 78.74 0)
       (effects (font (size 1.27 1.27)) hide)
     )
@@
       (effects (font (size 1.27 1.27)))
     )
-    (property "Footprint" "Connector_PinHeader_1.00mm:PinHeader_1x26_P1.00mm_Vertical" (at 93.98 176.53 0)
+    (property "Footprint" "Connector_PinHeader_2.54mm:PinHeader_1x26_P2.54mm_Vertical" (at 93.98 176.53 0)
       (effects (font (size 1.27 1.27)) hide)
     )
@@
       (effects (font (size 1.27 1.27)))
     )
-    (property "Footprint" "Connector_PinHeader_1.00mm:PinHeader_1x08_P1.00mm_Vertical" (at 207.01 80.01 0)
+    (property "Footprint" "Connector_PinHeader_2.54mm:PinHeader_1x08_P2.54mm_Vertical" (at 207.01 80.01 0)
       (effects (font (size 1.27 1.27)) hide)
     )
@@
       (effects (font (size 1.27 1.27)))
     )
-    (property "Footprint" "Connector_PinHeader_1.00mm:PinHeader_1x08_P1.00mm_Vertical" (at 20.32 77.47 0)
-      (effects (font (size 1.27 1.27)) hide)
-    )
+    (property "Footprint" "Connector_PinHeader_2.54mm:PinHeader_1x08_P2.54mm_Vertical" (at 20.32 77.47 0)
+      (effects (font (size 1.27 1.27)) hide)
+    )

Commit message: Updates v1.0
Parts:
- added J10: Conn_01x05_Socket, Connector_PinSocket_2.00mm:PinSocket_1x05_P2.00mm_Vertical, symbol Connector:Conn_01x05_Socket
- added J11: Conn_01x17_Socket, Connector_PinSocket_2.00mm:PinSocket_1x17_P2.00mm_Vertical, symbol Connector:Conn_01x17_Socket
- added J12: Conn_01x04_Socket, Connector_PinSocket_2.00mm:PinSocket_1x04_P2.00mm_Vertical, symbol Connector:Conn_01x04_Socket
- added J7, J8: Conn_01x05_Pin, Connector_PinHeader_2.54mm:PinHeader_1x05_P2.54mm_Vertical, symbol Connector:Conn_01x05_Pin
- added J9: Conn_01x06_Pin, Connector_PinHeader_2.54mm:PinHeader_1x06_P2.54mm_Vertical, symbol Connector:Conn_01x06_Pin
Connections:
- net at Q8.1: now also Q1.1, Q10.1, Q11.1, Q12.1, Q13.1, Q14.1, Q15.1, Q16.1, Q17.1, Q18.1, Q19.1, Q2.1, Q20.1, Q21.1, Q22.1, Q23.1, Q24.1, Q25.1, Q26.1, Q27.1, Q28.1, Q29.1, Q3.1, Q30.1, Q31.1, Q32.1, Q4.1, Q5.1, Q6.1, Q7.1, Q9.1, J7.5 (Pin_5), J8.5 (Pin_5), J9.6 (Pin_6); no longer J1.8 (Pin_8)
- net at J5.8 (Pin_8), Q8.4: now also J11.3 (Pin_3)
- net at J3.7 (Pin_7): now also Q23.2; no longer Q23.1
- net at J5.23 (Pin_23), Q23.4: now also J12.1 (Pin_1)
- net at J2.3 (Pin_3): now also Q11.2; no longer Q11.1
- net at J5.11 (Pin_11), Q11.4: now also J11.6 (Pin_6)
- net at J4.5 (Pin_5): now also Q29.2; no longer Q29.1
- net at J3.1 (Pin_1): now also Q17.2; no longer Q17.1
- net at J5.17 (Pin_17), Q17.4: now also J11.12 (Pin_12)
- net at J3.8 (Pin_8): now also Q24.2; no longer Q24.1
- net at J5.24 (Pin_24), Q24.4: now also J12.2 (Pin_2)
- net at J3.6 (Pin_6): now also Q22.2; no longer Q22.1
- net at J5.22 (Pin_22), Q22.4: now also J11.17 (Pin_17)
- net at J3.3 (Pin_3): now also Q19.2; no longer Q19.1
- net at J5.19 (Pin_19), Q19.4: now also J11.14 (Pin_14)
- net at J3.5 (Pin_5): now also Q21.2; no longer Q21.1
- net at J5.21 (Pin_21), Q21.4: now also J11.16 (Pin_16)
- net at J4.2 (Pin_2): now also Q26.2; no longer Q26.1
- net at J5.26 (Pin_26), Q26.4: now also J12.4 (Pin_4)
- net at J1.7 (Pin_7): now also Q7.2; no longer Q7.1
- net at J5.7 (Pin_7), Q7.4: now also J11.2 (Pin_2)
- net at J2.1 (Pin_1): now also Q9.2; no longer Q9.1
- net at J2.2 (Pin_2): now also Q10.2; no longer Q10.1
- net at J2.4 (Pin_4): now also Q12.2; no longer Q12.1
- net at J2.5 (Pin_5): now also Q13.2; no longer Q13.1
- net at J2.6 (Pin_6): now also Q14.2; no longer Q14.1
- net at J2.7 (Pin_7): now also Q15.2; no longer Q15.1
- net at J2.8 (Pin_8): now also Q16.2; no longer Q16.1
- net at J1.4 (Pin_4): now also Q4.2; no longer Q4.1
- net at J5.4 (Pin_4), Q4.4: now also J10.4 (Pin_4)
- net at J4.4 (Pin_4): now also Q28.2; no longer Q28.1
- net at J4.1 (Pin_1): now also Q25.2; no longer Q25.1
- net at J5.25 (Pin_25), Q25.4: now also J12.3 (Pin_3)
- net at J3.2 (Pin_2): now also Q18.2; no longer Q18.1
- net at J3.4 (Pin_4): now also Q20.2; no longer Q20.1
- net at J5.15 (Pin_15), Q15.4: now also J11.10 (Pin_10)
- net at J5.14 (Pin_14), Q14.4: now also J11.9 (Pin_9)
- net at J4.8 (Pin_8): now also Q32.2; no longer Q32.1
- net at J4.3 (Pin_3): now also Q27.2; no longer Q27.1
- net at J5.10 (Pin_10), Q10.4: now also J11.5 (Pin_5)
- net at J5.18 (Pin_18), Q18.4: now also J11.13 (Pin_13)
- net at J5.16 (Pin_16), Q16.4: now also J11.11 (Pin_11)
- net at J5.20 (Pin_20), Q20.4: now also J11.15 (Pin_15)
- net at J1.3 (Pin_3): now also Q3.2; no longer Q3.1
- net at J5.3 (Pin_3), Q3.4: now also J10.3 (Pin_3)
- net at J5.1 (Pin_1), Q1.4: now also J10.1 (Pin_1)
- net at J5.12 (Pin_12), Q12.4: now also J11.7 (Pin_7)
- net at J5.13 (Pin_13), Q13.4: now also J11.8 (Pin_8)
- net at J5.2 (Pin_2), Q2.4: now also J10.2 (Pin_2)
- net at J5.5 (Pin_5), Q5.4: now also J10.5 (Pin_5)
- net at J5.6 (Pin_6), Q6.4: now also J11.1 (Pin_1)
- net at J5.9 (Pin_9), Q9.4: now also J11.4 (Pin_4)
- net at J1.2 (Pin_2): now also Q2.2; no longer Q2.1
- net at J1.1 (Pin_1): now also Q1.2; no longer Q1.1
- net at J1.5 (Pin_5): now also Q5.2; no longer Q5.1
- net at J4.7 (Pin_7): now also Q31.2; no longer Q31.1
- net at J4.6 (Pin_6): now also Q30.2; no longer Q30.1
- net at J1.6 (Pin_6): now also Q6.2; no longer Q6.1
- new net: J7.1 (Pin_1), J8.1 (Pin_1), J9.1 (Pin_1)
- new net: J8.2 (Pin_2), J9.3 (Pin_3)
- new net: J7.3 (Pin_3), J8.3 (Pin_3), J9.4 (Pin_4)
- new net: J7.4 (Pin_4), J8.4 (Pin_4), J9.5 (Pin_5)
- new net: J1.8 (Pin_8), Q8.2
- new net: J7.2 (Pin_2), J9.2 (Pin_2)
